File: A3-Flight-Computer-Hardware/A3-Flight-Computer-Hardware.kicad_sch (KiCad schematic)
At the start: 28 parts, among them J1 Micro_SD_Card, J2 Telem, J3 USB_C_Receptacle_USB2.0_14P, J4 Cam 1, J5 Cam 2, J6 CAN, J7 Cam 3, U2 PTCAN3414DR, U3 ADXL375BCCZ-RL7, U4 LPS22HBTR, U5 LSM6DSO32TR, U6 AP2112K-3.3TRG1, U7 STM32H523RETx, Y1 TSX-3225_16.0000MF18X-AC0, Y2 ECS-.327-9-34QCS-TR

Commit message: Initial schematic
Parts:
- removed C1: 4.7nF, Capacitor_SMD:C_0805_2012Metric, symbol Device:C_Small_US
- removed D1, D2: SMF54CA, Diode_SMD:D_SMF, symbol Diode:SMAJ54CA
- removed J1: Micro_SD_Card, Connector_Card:microSD_HC_Molex_47219-2001, symbol Connector:Micro_SD_Card
- removed J2: Telem, Connector_JST:JST_XH_S2B-XH-A_1x02_P2.50mm_Horizontal, symbol Connector:Conn_01x02_Pin
- removed J6: CAN, Connector_JST:JST_XH_S2B-XH-A_1x02_P2.50mm_Horizontal, symbol Connector:Conn_01x02_Pin
- removed R3, R4: 60, Resistor_SMD:R_0805_2012Metric, symbol Device:R_Small_US
- removed U2: PTCAN3414DR, A3-Flight-Computer:SOIC8_D_TEX, symbol A3-Flight-Computer-Components:PTCAN3414DR
- removed U3: ADXL375BCCZ-RL7, A3-Flight-Computer:LGA_CC-14-1_ADI, symbol A3-Flight-Computer-Components:ADXL375BCCZ-RL7
- removed U4: LPS22HBTR, A3-Flight-Computer:PQFN50P200X200X80-10N, symbol A3-Flight-Computer-Components:LPS22HBTR
- removed U5: LSM6DSO32TR, A3-Flight-Computer:XDCR_LSM6DSO32TR, symbol A3-Flight-Computer-Components:LSM6DSO32TR
- removed U6: AP2112K-3.3TRG1, A3-Flight-Computer:SOT95P285X140-5N, symbol A3-Flight-Computer-Components:AP2112K-3.3TRG1
- added C15, C16: 2.2uF, Capacitor_SMD:C_0805_2012Metric, symbol Device:C_Small_US
- added C17, C18, C19, C20, C21, C23, C3: 100nF, Capacitor_SMD:C_0805_2012Metric, symbol Device:C_Small_US
- added C22: 4.7uF, Capacitor_SMD:C_0805_2012Metric, symbol Device:C_Small_US
- added D1, D2: DSS14U, Diode_SMD:D_SOD-123, symbol Diode:BAV16W
- added D6, D7: LED, LED_SMD:LED_0805_2012Metric_Pad1.15x1.40mm_HandSolder, symbol Device:LED
- added J1: BAT, Connector_JST:JST_XH_S2B-XH-A_1x02_P2.50mm_Horizontal, symbol Connector:Conn_01x02_Pin
- added J2: ST1W008S4ER1500, A3-Flight-Computer:JAE_ST1W008S4ER1500, symbol A3-Flight-Computer-Components:ST1W008S4ER1500
- added J5: Debug Header, Connector_PinSocket_2.54mm:PinSocket_2x03_P2.54mm_Vertical, symbol Connector_Generic:Conn_02x03_Top_Bottom
- added J8: Telem, Connector_JST:JST_XH_S2B-XH-A_1x02_P2.50mm_Horizontal, symbol Connector:Conn_01x02_Pin
- added R7: 10k, LED_SMD:LED_0805_2012Metric, symbol Device:R_Small_US
- added R8, R9: 240R, LED_SMD:LED_0805_2012Metric, symbol Device:R_Small_US
- added SW1: BOOT, Button_Switch_SMD:SW_DIP_SPSTx01_Slide_Copal_CVS-01xB_W5.9mm_P1mm, symbol Switch:SW_SPDT
- added SW2: RST, Button_Switch_SMD:SW_SPST_EVQPE1, symbol Switch:SW_Push
- added VR1: AZ1117CH-3.3TRG1, A3-Flight-Computer:VREG_AZ1117CH-3.3TRG1, symbol A3-Flight-Computer-Components:AZ1117CH-3.3TRG1
- C1: renamed from C7; value 1uF -> 22uF
- C2: renamed from C6; value 1uF -> 10uF
- C4: renamed from C2; value 3pF -> 8pF
- C5: renamed from C3; value 3pF -> 8pF
- renumbered C4 to C6, C5 to C7, J5 to J6, U7 to U1
Connections:
- net +3.3V: now also U1.1 (VBAT), U1.13 (VDDA), U1.19 (VDD), U1.32 (VDD), U1.48 (VDD), U1.64 (VDD), C17.1, C18.1, C19.1, C20.1, C21.1, C22.1, C3.1, D6.2 (A), J2.4 (VDD), SW1.1 (A), VR1.2 (OUTPUT), VR1.4 (OUTPUT__1)
- net CAM1_RX: now also J4.2 (Pin_2)
- net CAM1_TX: now also J4.1 (Pin_1)
- net CAM2_RX: now also J6.2 (Pin_2)
- net CAM2_TX: now also J6.1 (Pin_1)
- net CAM3_RX: now also J7.2 (Pin_2)
- net CAM3_TX: now also J7.1 (Pin_1)
- net DEBUG_RX: now also U1.58 (PB6), J5.6 (Pin_6); no longer U1.59 (PB7)
- net DEBUG_TX: now also U1.57 (PB5), J5.3 (Pin_3); no longer U1.58 (PB6)
- net GND: now also C15.2, C16.2, C17.2, C18.2, C19.2, C20.2, C21.2, C22.2, C23.2, C3.2, J1.2 (Pin_2), J2.6 (VSS), J2.GND1 (GND), J2.GND2 (GND__1), J2.GND3 (GND__2), J2.GND4 (GND__3), R8.1, R9.1, SW1.3 (C), SW2.1, VR1.1 (GND)
- net JTCK-SWCLK: now also J5.4 (Pin_4)
- net JTDI: now also J5.5 (Pin_5)
- net JTDO-SWO: now also J5.2 (Pin_2)
- net JTMS-SWDIO: now also J5.1 (Pin_1)
- net SD_CK: now also J2.5 (CLK)
- net SD_CMD: now also J2.3 (CMD)
- net SD_D0: now also J2.7 (DAT0)
- net SD_D1: now also J2.8 (DAT1)
- net SD_D2: now also J2.1 (DAT2)
- net SD_D3: now also J2.2 (DAT3/CD)
- net TELEM_RX: now also J8.2 (Pin_2)
- net TELEM_TX: now also J8.1 (Pin_1)
- net at J3.A4 (VBUS), J3.A9 (VBUS), J3.B4 (VBUS)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: now also D2.2 (A); no longer C2.1
- net ADXL375_INT1: now reaches U1.20 (PA4)
- net ADXL375_INT2: now reaches U1.21 (PA5)
- net LSM6_INT1: now reaches U1.22 (PA6)
- net LSM6_INT2: now reaches U1.23 (PA7)
- net CAN_STBD: now reaches U1.24 (PC4)
- net CAN_SHD: now reaches U1.25 (PC5)
- net LPS22HB_INT: now reaches U1.26 (PB0)
- net STAT_LED: now reaches U1.28 (PB2)
- net STAT_LED: now also D7.2 (A)
- net at U1.30 (VCAP): now also U1.62 (VCAP), C15.1, C16.1
- net I2C_SCL: now reaches U1.41 (PA8)
- net I2C_SDA: now reaches U1.56 (PB4(NJTRST))
- net BOOT: now reaches U1.60 (BOOT0)
- net BOOT: now also R7.2
- net RST: now reaches U1.7 (NRST)
- net RST: now also C23.1, SW2.2
- new net: C2.1, D1.1 (K), D2.1 (K), VR1.3 (INPUT)
- new net: D1.2 (A), J1.1 (Pin_1)
- new net: R7.1, SW1.2 (B)
- new net: D7.1 (K), R9.2
- new net: D6.1 (K), R8.2
- no-connect marks 0 -> 11
Other:
- added sheet Peripheral Devices (peripheral.kicad_sch)
- moved on the sheet: C1, C2, C4, C5, C6, C7, J3, J4, J6, J7, R1, R2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

Commit message: First PCB revision
Parts:
- added BZ1: Buzzer, Buzzer_Beeper:Buzzer_Murata_PKMCS0909E, symbol Device:Buzzer
- added D5: SS14, Diode_SMD:D_SMA, symbol Diode:SS14
- added Q1: IRLML0030, Package_TO_SOT_SMD:SOT-23, symbol Transistor_FET:IRLML0030
- added R3, R4: 27R, Resistor_SMD:R_0805_2012Metric, symbol Device:R_Small_US
- added R8: 100, Resistor_SMD:R_0805_2012Metric, symbol Device:R_Small_US
- added R9: 100k, Resistor_SMD:R_0805_2012Metric, symbol Device:R_Small_US
- C14: renamed from C6; value 4pF -> 16pF
- C15: renamed from C7; value 4pF -> 16pf
- J4: renamed from J5; footprint Connector_PinSocket_2.54mm:PinSocket_2x03_P2.54mm_Vertical -> Connector_PinHeader_2.54mm:PinHeader_2x03_P2.54mm_Vertical
- J8: footprint Connector_JST:JST_XH_S2B-XH-A_1x02_P2.50mm_Horizontal -> Connector_JST:JST_XH_S3B-XH-A_1x03_P2.50mm_Horizontal; symbol Connector:Conn_01x02_Pin -> Connector:Conn_01x03_Pin
- R5: renamed from R8; footprint LED_SMD:LED_0805_2012Metric -> Resistor_SMD:R_0805_2012Metric
- R6: renamed from R7; footprint LED_SMD:LED_0805_2012Metric -> Resistor_SMD:R_0805_2012Metric
- R7: renamed from R9; footprint LED_SMD:LED_0805_2012Metric -> Resistor_SMD:R_0805_2012Metric
- SW1: footprint Button_Switch_SMD:SW_DIP_SPSTx01_Slide_Copal_CVS-01xB_W5.9mm_P1mm -> Button_Switch_SMD:SW_SPDT_CK_JS102011SAQN
- SW2: footprint Button_Switch_SMD:SW_SPST_EVQPE1 -> Button_Switch_SMD:SW_SPST_TS-1088-xR025
- renumbered C22 to C1, C4 to C10, C5 to C11, C16 to C12, C15 to C13, C23 to C16, C17 to C2, C18 to C3, C19 to C4, C20 to C5, C21 to C6, C1 to C7, C2 to C8, C3 to C9, D6 to D3, D7 to D4, J4 to J5
Connections:
- net +3.3V: now also BZ1.1 (+), D5.1 (K)
- net ADXL375_INT1: now also U1.21 (PA5); no longer U1.20 (PA4)
- net ADXL375_INT2: now also U1.20 (PA4); no longer U1.21 (PA5)
- net DEBUG_RX: now also J4.5 (Pin_5); no longer J4.6 (Pin_6)
- net DEBUG_TX: now also J4.6 (Pin_6); no longer J4.3 (Pin_3)
- net GND: now also J8.3 (Pin_3), Q1.2 (S), R9.1
- net JTDI: now also J4.3 (Pin_3); no longer J4.5 (Pin_5)
- net JTDO-SWO: now also J4.1 (Pin_1); no longer J4.2 (Pin_2)
- net JTMS-SWDIO: now also J4.2 (Pin_2); no longer J4.1 (Pin_1)
- net USB_DM: now also R3.1; no longer J3.A7 (D-), J3.B7 (D-)
- net USB_DP: now also R4.1; no longer J3.A6 (D+), J3.B6 (D+)
- net BUZZ: now reaches U1.35 (PB14)
- net BUZZ: now also R8.1
- new net: BZ1.2 (-), D5.2 (A), Q1.3 (D)
- new net: J3.A6 (D+), J3.B6 (D+), R4.2
- new net: J3.A7 (D-), J3.B7 (D-), R3.2
- new net: Q1.1 (G), R8.2, R9.2
- no-connect marks 11 -> 10
Other:
- moved on the sheet: J4
