File: A3-Flight-Computer-Hardware/A3-Flight-Computer-Hardware-Rectangular.kicad_sch (KiCad schematic)
At the start: 45 parts, among them J1 BAT, J2 ST1W008S4ER1500, J3 USB_C_Receptacle_USB2.0_14P, J4 Debug Header, J5 Cam 1, J6 Cam 2, J8 Telem, Q1 IRLML0030, SW1 BOOT, SW2 RST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

Commit message: Small routing changes
Parts:
- removed J4: Debug Header, Connector_PinHeader_2.54mm:PinHeader_2x03_P2.54mm_Vertical, symbol Connector_Generic:Conn_02x03_Top_Bottom
- added J4: Conn_02x04_Odd_Even, Connector_PinHeader_2.54mm:PinHeader_2x04_P2.54mm_Vertical, symbol Connector_Generic:Conn_02x04_Odd_Even
Connections:
- net +3.3V: now also J4.2 (Pin_2)
- net DEBUG_RX: now also J4.8 (Pin_8)
- net DEBUG_TX: now also J4.7 (Pin_7)
- net GND: now also J4.1 (Pin_1)
- net JTCK-SWCLK: now also J4.5 (Pin_5)
- net JTDI: now also J4.4 (Pin_4)
- net JTDO-SWO: now also J4.3 (Pin_3)
- net JTMS-SWDIO: now also J4.6 (Pin_6)

Commit message: Added labels and changed component sizes
Parts:
- removed D5: SS14, Diode_SMD:D_SMA, symbol Diode:SS14
- added C7: 100nF, Capacitor_SMD:C_0402_1005Metric, symbol Device:C_Small_US
- added D4: LED, LED_SMD:LED_0805_2012Metric_Pad1.15x1.40mm_HandSolder, symbol Device:LED
- added D6: DSS14U, Diode_SMD:D_SOD-123, symbol Diode:BAV16W
- added R7: 240R, Resistor_SMD:R_0402_1005Metric, symbol Device:R_Small_US
- C10: renamed from C9; footprint Capacitor_SMD:C_0805_2012Metric -> Capacitor_SMD:C_0402_1005Metric
- C11: renamed from C10; footprint Capacitor_SMD:C_0805_2012Metric -> Capacitor_SMD:C_0402_1005Metric
- C12: renamed from C11; footprint Capacitor_SMD:C_0805_2012Metric -> Capacitor_SMD:C_0402_1005Metric
- C13: renamed from C12; footprint Capacitor_SMD:C_0805_2012Metric -> Capacitor_SMD:C_0402_1005Metric
- C14: renamed from C13; footprint Capacitor_SMD:C_0805_2012Metric -> Capacitor_SMD:C_0402_1005Metric
- C15: renamed from C14; footprint Capacitor_SMD:C_0805_2012Metric -> Capacitor_SMD:C_0402_1005Metric
- C16: renamed from C15; footprint Capacitor_SMD:C_0805_2012Metric -> Capacitor_SMD:C_0402_1005Metric
- C17: renamed from C16; footprint Capacitor_SMD:C_0805_2012Metric -> Capacitor_SMD:C_0402_1005Metric
- C2, C3, C4, C5, C6: footprint Capacitor_SMD:C_0805_2012Metric -> Capacitor_SMD:C_0402_1005Metric
- J4: renamed from J5; footprint Connector_JST:JST_XH_B2B-XH-A_1x02_P2.50mm_Vertical -> Connector_JST:JST_XH_S2B-XH-A_1x02_P2.50mm_Horizontal
- J5: renamed from J4; value Conn_02x04_Odd_Even -> DEBUG
- J6: footprint Connector_JST:JST_XH_B2B-XH-A_1x02_P2.50mm_Vertical -> Connector_JST:JST_XH_S2B-XH-A_1x02_P2.50mm_Horizontal
- J7: renamed from J8; footprint Connector_JST:JST_XH_B3B-XH-A_1x03_P2.50mm_Vertical -> Connector_JST:JST_XH_S3B-XH-A_1x03_P2.50mm_Horizontal
- R1, R2, R3, R4, R5, R6: footprint Resistor_SMD:R_0805_2012Metric -> Resistor_SMD:R_0402_1005Metric
- R10: renamed from R9; footprint Resistor_SMD:R_0805_2012Metric -> Resistor_SMD:R_0402_1005Metric
- R8: renamed from R7; footprint Resistor_SMD:R_0805_2012Metric -> Resistor_SMD:R_0402_1005Metric
- R9: renamed from R8; footprint Resistor_SMD:R_0805_2012Metric -> Resistor_SMD:R_0402_1005Metric
- renumbered C7 to C8, C8 to C9, D4 to D5
Connections:
- net +3.3V: now also C7.1, D6.1 (K)
- net BUZZ: now also U1.24 (PC4); no longer U1.10 (PC2)
- net CAN_SHD: now also U1.35 (PB14); no longer U1.25 (PC5)
- net CAN_STBD: now also U1.36 (PB15); no longer U1.24 (PC4)
- net GND: now also C7.2, R7.1
- net at BZ1.2 (-), Q1.3 (D): now also D6.2 (A)
- net STAT_LED1: now reaches U1.27 (PB1)
- net STAT_LED1: now also D4.2 (A)
- net STAT_LED renamed STAT_LED2
- new net: D4.1 (K), R7.2
- no-connect marks 14 -> 11
Other:
- note added: "MircoSD Interface"
- moved on the sheet: BZ1, D5, J4, J6, J7, Q1, R10, R8, R9
