File: A3-Flight-Computer-Hardware/peripheral.kicad_sch (KiCad schematic)
At the start: 18 parts, among them J9 CAN, U2 ADXL375BCCZ-RL7, U3 LSM6DSO32TR, U4 LPS22HBTR, U5 PTCAN3414DR

Commit message: First PCB revision
Parts:
- renumbered C10 to C17, C11 to C18, C8 to C19, C9 to C20, C12 to C21, C13 to C22, C14 to C23, D3 to D6, D4 to D7, R3 to R10, R4 to R11, R5 to R12, R6 to R13

Commit message: Adjusted PCB Dimensions
Parts:
- added C23: 100nF, Capacitor_SMD:C_0805_2012Metric, symbol Device:C_Small_US
- renumbered C23 to C24
Connections:
- net +3.3V: now also C23.1
- net GND: now also C23.2

Commit message: Added labels and changed component sizes
Parts:
- added TP3: SDA, TestPoint:TestPoint_THTPad_1.0x1.0mm_Drill0.5mm, symbol Connector:TestPoint
- added TP4: SCL, TestPoint:TestPoint_THTPad_1.0x1.0mm_Drill0.5mm, symbol Connector:TestPoint
- C18: renamed from C17; footprint Capacitor_SMD:C_0805_2012Metric -> Capacitor_SMD:C_0402_1005Metric
- C19: renamed from C18; footprint Capacitor_SMD:C_0805_2012Metric -> Capacitor_SMD:C_0402_1005Metric
- C20: renamed from C19; footprint Capacitor_SMD:C_0805_2012Metric -> Capacitor_SMD:C_0402_1005Metric
- C21: renamed from C20; footprint Capacitor_SMD:C_0805_2012Metric -> Capacitor_SMD:C_0402_1005Metric
- C22: renamed from C21; footprint Capacitor_SMD:C_0805_2012Metric -> Capacitor_SMD:C_0402_1005Metric
- C23: renamed from C22; footprint Capacitor_SMD:C_0805_2012Metric -> Capacitor_SMD:C_0402_1005Metric
- C24: renamed from C23; footprint Capacitor_SMD:C_0805_2012Metric -> Capacitor_SMD:C_0402_1005Metric
- C25: renamed from C24; footprint Capacitor_SMD:C_0805_2012Metric -> Capacitor_SMD:C_0402_1005Metric
- R11: renamed from R10; footprint Resistor_SMD:R_0805_2012Metric -> Resistor_SMD:R_0402_1005Metric
- R12: renamed from R11; footprint Resistor_SMD:R_0805_2012Metric -> Resistor_SMD:R_0402_1005Metric
- R13: renamed from R12; footprint Resistor_SMD:R_0805_2012Metric -> Resistor_SMD:R_0402_1005Metric
- R14: renamed from R13; footprint Resistor_SMD:R_0805_2012Metric -> Resistor_SMD:R_0402_1005Metric
- renumbered D6 to D7, D7 to D8, J9 to J8
Connections:
- net SCL: now also TP4.1
- net SDA: now also TP3.1
Other:
- note added: "Accelerometer (+/- 200g) I2C Address: 0x53 (0b1010011)"
- note added: "Accelerometer/Gyroscope (+/- 32g) I2C Address: 0x6A (0b1101010)"
- note added: "Temperature/Pressure I2C Address: 0x5C (0b1011100)"
